Commit message: feat: add ros2_control omni base controller

File: qianli_ws/src/qianli_description/urdf/base.xacro (robot description, xacro)
@@ -2,6 +2,9 @@
 <robot xmlns:xacro="http://www.ros.org/wiki/xacro">
   <xacro:macro name="qianli_base" params="">
-    <link name="base_footprint"/>
+    <link name="base_footprint">
+      <xacro:if value="${simulation}"><xacro:sim_frame_inertial/></xacro:if>
+    </link>
     <link name="base_link">
+      <xacro:if value="${simulation}"><xacro:sim_plate_inertial/></xacro:if>
       <visual name="octagonal_plate">
         <geometry><mesh filename="package://qianli_description/meshes/base/qianli_base.stl"/></geometry>

File: qianli_ws/src/qianli_description/urdf/qianli.urdf.xacro (robot description, xacro)
@@ -1,8 +1,17 @@
 <?xml version="1.0"?>
 <robot name="qianli" xmlns:xacro="http://www.ros.org/wiki/xacro">
+  <xacro:arg name="control_mode" default="none"/>
+  <xacro:arg name="controllers_file" default=""/>
+  <xacro:arg name="simulation" default="false"/>
+  <xacro:property name="simulation" value="$(arg simulation)"/>
   <xacro:include filename="common.xacro"/>
   <xacro:include filename="base.xacro"/>
   <xacro:include filename="wheels.xacro"/>
+  <xacro:include filename="ros2_control.xacro"/>
+  <xacro:include filename="sim_inertials.xacro"/>
   <xacro:qianli_base/>
   <xacro:qianli_wheels/>
+  <xacro:if value="${'$(arg control_mode)' != 'none'}">
+    <xacro:qianli_control mode="$(arg control_mode)" controllers_file="$(arg controllers_file)"/>
+  </xacro:if>
 </robot>

File: qianli_ws/src/qianli_description/urdf/wheels.xacro (robot description, xacro)
@@ -3,4 +3,5 @@
   <xacro:macro name="qianli_wheel" params="name x_sign y_sign yaw">
     <link name="${name}_wheel_link">
+      <xacro:if value="${simulation}"><xacro:sim_wheel_inertial/></xacro:if>
       <!-- Cylinder axis and joint axis are both local +Z. -->
       <visual>
