Commit message: feat(arm): 在模型里定义 TCP + 实测桌面高度（含 FK 自检）
一、TCP 从模型算出并写进 URDF
- tcp_from_model.py：把两爪"最接近处"当作抓取点求解。第一版把整个 gripper_link
  外壳都算进去，最近点落在**铰链**（frame z=-74mm）而不是夹取面，加
  --front-mm 限制到爪尖前端 25mm 后才正确。
- 结果：固定爪内侧面落在 gripper_frame_link 的 X≈0，开口中心 = X0 - W/2，
  Z 取两爪接触深度。按 14mm 物块 → TCP = (-7.00, 0, +2.37) mm。
- 重要更正：**上一轮"TCP 比爪口低 3.4cm"的结论是错的。** 实测 TCP 距爪尖
  只有 4.6mm，整轮抓空的解释需要重查。那个 9.81cm 恰好等于
  gripper_frame_joint 的偏置 98.1mm，说明当时参照取错了。
- tcp_link 挂为 gripper_frame_link 的子节点，ikpy 链末端自动变成 tcp_joint，
  IK 从此直接解算抓取点。tool_pose / calib_grasp_offset / extrinsic_calib
  里的参考坐标系同步改为 tcp_link。
- hardware/mechanical_arm/docs/tcp_grasp_point.png：渲染图，红色方块是
  14mm 物块，正好卡在两爪之间。

二、桌面实测（取代旧假设）
- 发现关键概念错误：**碰到桌面的是"夹爪几何最低点"，不是 TCP。**
  tcp_offset_sweep 实测：TCP 相对最低点的高度随姿态从 +5.1mm 变到 +100.6mm
  （跨度 95.5mm）。所以"让爪子碰桌子读 TCP 的 Z"读数必然漂移 —— 第一次
  用 TCP 采 6 点相差 31mm，改用最低点后只差 1.5mm。
- table_limit_gui.py：网页前端，实时显示模型算出的夹爪最低点，人工点确认。
- 结果：桌面 -69.09mm，平面倾角 0.202°，拟合残差 RMS 0.469mm（6 点，
  跨度 239x353mm，姿态各异）→ 残差本身就是对 FK 的验证。
- **旧假设 board_z=-49.4mm 偏高了 19.7mm**，需要重算抓取下压深度。
- safe_z_min = -60.48mm。

三、FK 自检（两个静默 bug 被抓出）
- ikpy 的 link.name 是**关节名**不是 URDF link 名，按 link 名取值全部取不到、
  静默退化成"整条链的乘积"。
- forward_kinematics(full_kinematics=True) 返回的每项**已经是 base→link 的
  累积变换**，再累乘一次会让所有位姿都错 —— 但数值看起来正常、不报错。
- gripper_model.GripperModel.selftest() 专门盯这类退化：比较 gripper_link 与
  tcp_link 是否重合、tcp_link 是否满足固定偏移、活动爪是否真随关节动。
- 另外修掉 NumPy 2.0 已移除的 ndarray.ptp()（导致前端 plane 恒为 null）。

File: qianli_ws/src/qianli_description/urdf/so101.urdf (robot description, URDF)
Before this commit: robot so101_new_calib, 8 links, 7 joints
Links:
- added link tcp_link, mass 1e-9
Joints:
- added joint tcp_joint: type fixed, parent gripper_frame_link, child tcp_link, origin xyz=-0.007000 0.000000 0.002373 rpy=0 0 0, axis 0 0 0
